File: Schematics/HV_DISTRUBUTIONN/HV-DST.brd (EAGLE design)
At the start: 100 x 80 mm, 40 parts

Commit message: Working on layout for distribution
Parts:
- removed C1, C3, C5, C7: 330pF, capacitor-wima:C2.5-2
- added SV1: (no value), con-lsta:FE05-1
- moved U$4 82.7 mm to (5.08, 61.0), turned to 270 degrees
- moved R6 81.4 mm to (24.1, 27.9), turned to 180 degrees
- moved U$5 78.5 mm to (27.9, 74.9), turned to 180 degrees
- moved R12 75.0 mm to (17.8, 34.3)
- moved R10 70.0 mm to (24.1, 44.5), turned to 180 degrees
- moved R16 63.5 mm to (17.8, 50.8)
- moved U$3 63.3 mm to (5.08, 44.5), turned to 270 degrees
- moved C9 60.7 mm to (26.7, 66.0)
- moved R14 60.4 mm to (24.1, 61.0), turned to 180 degrees
- moved R4 54.0 mm to (17.8, 1.27)
- moved R3 44.7 mm to (24.1, 11.4), turned to 180 degrees
- moved U$2 44.4 mm to (5.08, 27.9), turned to 270 degrees
- moved R8 39.0 mm to (17.8, 17.8)
- moved U$1 27.4 mm to (5.08, 11.4), turned to 270 degrees
Connections:
- net G1: now also SV1.1
- net G2: now also SV1.2
- net G3: now also SV1.3
- net G4: now also SV1.4
- net GND: now also SV1.5; no longer C1.2, C3.2, C5.2, C7.2
- net N$10: no longer C5.1
- net N$14: no longer C7.1
- net N$2: no longer C1.1
- net N$6: no longer C3.1
Routing:
- net V+: track 0.00 -> 73.7 mm
- net N$14: track 0.00 -> 14.0 mm
- net GND: track 0.00 -> 9.94 mm
- net N$16: track 0.00 -> 9.16 mm
- net N$4: track 0.00 -> 9.16 mm
- net N$8: track 0.00 -> 9.16 mm
- net N$12: track 0.00 -> 9.16 mm

Commit message: Finished routing
Parts:
- added R19, R20, R21, R22: 100, resistor-power:RS1/4
- moved R17 136.6 mm to (78.7, 24.1), turned to 270 degrees
- moved IC1 118.4 mm to (76.2, 24.1), turned to 270 degrees
- moved SV1 117.2 mm to (57.1, 5.08), turned to 180 degrees
- moved R11 108.6 mm to (45.7, 47.0)
- moved U$6 102.1 mm to (68.6, 3.81)
- moved C8 101.8 mm to (40.6, 59.7), turned to 270 degrees
- moved C10 101.7 mm to (72.4, 15.2), turned to 180 degrees
- moved T4 100.4 mm to (35.6, 61.0), turned to 270 degrees
- moved C11 99.8 mm to (64.8, 22.9), turned to 270 degrees
- moved R7 99.3 mm to (45.7, 30.5)
- moved R1 93.8 mm to (45.7, 14.0)
- moved R18 91.5 mm to (69.8, 24.1), turned to 90 degrees
- moved T3 91.4 mm to (35.6, 44.5), turned to 270 degrees
- moved C6 89.5 mm to (40.6, 43.2), turned to 270 degrees
- moved R2 89.3 mm to (34.3, 5.08), turned to 180 degrees
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Connections:
- new net N$15: R20.2, SV1.2
- new net N$17: R21.2, SV1.3
- new net N$18: R22.2, SV1.4
- new net N$7: R19.2, SV1.1
- net G1: now also R22.1; no longer SV1.1
- net G2: now also R21.1; no longer SV1.2
- net G3: now also R20.1; no longer SV1.3
- net G4: now also R19.1; no longer SV1.4
Routing:
- net GND: track 9.94 -> 185.2 mm
- net +3V3: track 0.00 -> 149.0 mm
- net N$7: track 0.00 -> 68.7 mm
- net N$15: track 0.00 -> 51.1 mm
- net N$17: track 0.00 -> 32.8 mm
- net N$3: track 0.00 -> 17.8 mm
- net N$18: track 0.00 -> 14.5 mm
- net N$6: track 0.00 -> 14.0 mm
- net N$2: track 0.00 -> 14.0 mm
- net N$10: track 0.00 -> 14.0 mm
- net N$9: track 0.00 -> 12.7 mm
- net N$5: track 0.00 -> 12.7 mm
- net N$13: track 0.00 -> 12.7 mm
- net N$1: track 0.00 -> 12.7 mm
- net N$11: track 0.00 -> 11.0 mm
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Other:
- board size 100 x 80 mm -> 82.2 x 81.3 mm
