File: Schematics/HV_DISTRUBUTIONN/HV-DST.sch (EAGLE design)
At the start: 40 parts

Commit message: Working on layout for distribution
Parts:
- removed C1, C3, C5, C7: 330pF, capacitor-wima:C2.5/2
- added SV1: (no value), con-lsta:FE05-1
Connections:
- net G1: now also SV1.1
- net G2: now also SV1.2
- net G3: now also SV1.3
- net G4: now also SV1.4
- net GND: now also SV1.5; no longer C1.2, C3.2, C5.2, C7.2
- net N$10: no longer C5.1
- net N$14: no longer C7.1
- net N$2: no longer C1.1
- net N$6: no longer C3.1
Changed lines of the file:
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@@
 <part name="R2" library="resistor-power" deviceset="R" device="RS1/4" value="100k"/>
 <part name="R3" library="resistor-power" deviceset="R" device="RS1/4" value="2.2k"/>
-<part name="C1" library="capacitor-wima" deviceset="C" device="2.5/2" value="330pF"/>
 <part name="C2" library="capacitor-wima" deviceset="C" device="2.5/2" value="330pF"/>
 <part name="R1" library="resistor-power" deviceset="R" device="RS1/4"/>
@@
 <part name="R5" library="resistor-power" deviceset="R" device="RS1/4" value="100k"/>
 <part name="R6" library="resistor-power" deviceset="R" device="RS1/4" value="2.2k"/>
-<part name="C3" library="capacitor-wima" deviceset="C" device="2.5/2" value="330pF"/>
 <part name="C4" library="capacitor-wima" deviceset="C" device="2.5/2" value="330pF"/>
 <part name="R7" library="resistor-power" deviceset="R" device="RS1/4"/>
@@
 <part name="R9" library="resistor-power" deviceset="R" device="RS1/4" value="100k"/>
 <part name="R10" library="resistor-power" deviceset="R" device="RS1/4" value="2.2k"/>
-<part name="C5" library="capacitor-wima" deviceset="C" device="2.5/2" value="330pF"/>
 <part name="C6" library="capacitor-wima" deviceset="C" device="2.5/2" value="330pF"/>
 <part name="R11" library="resistor-power" deviceset="R" device="RS1/4"/>
@@
 <part name="R13" library="resistor-power" deviceset="R" device="RS1/4" value="100k"/>
 <part name="R14" library="resistor-power" deviceset="R" device="RS1/4" value="2.2k"/>
-<part name="C7" library="capacitor-wima" deviceset="C" device="2.5/2" value="330pF"/>
 <part name="C8" library="capacitor-wima" deviceset="C" device="2.5/2" value="330pF"/>
 <part name="R15" library="resistor-power" deviceset="R" device="RS1/4"/>
@@
 <part name="U$6" library="muon-tube" deviceset="ED2609" device=""/>
 <part name="+3V5" library="supply1" deviceset="+3V3" device=""/>
+<part name="SV1" library="con-lsta" deviceset="FE05-1" device=""/>
+<part name="GND7" library="supply1" deviceset="GND" device=""/>
 </parts>
 <sheets>
@@
 <instance part="R2" gate="G$1" x="63.5" y="149.86" rot="R90"/>
 <instance part="R3" gate="G$1" x="63.5" y="165.1" rot="R90"/>
-<instance part="C1" gate="G$1" x="50.8" y="157.48"/>
 <instance part="C2" gate="G$1" x="81.28" y="154.94"/>
 <instance part="R1" gate="G$1" x="71.12" y="172.72" rot="R90"/>
@@
 <instance part="R5" gate="G$1" x="63.5" y="78.74" rot="R90"/>
 <instance part="R6" gate="G$1" x="63.5" y="93.98" rot="R90"/>
-<instance part="C3" gate="G$1" x="50.8" y="86.36"/>
 <instance part="C4" gate="G$1" x="81.28" y="83.82"/>
 <instance part="R7" gate="G$1" x="71.12" y="101.6" rot="R90"/>
@@
 <instance part="R9" gate="G$1" x="127" y="152.4" rot="R90"/>
 <instance part="R10" gate="G$1" x="127" y="167.64" rot="R90"/>
-<instance part="C5" gate="G$1" x="114.3" y="160.02"/>
 <instance part="C6" gate="G$1" x="144.78" y="157.48"/>
 <instance part="R11" gate="G$1" x="134.62" y="175.26" rot="R90"/>
@@
 <instance part="R13" gate="G$1" x="129.54" y="78.74" rot="R90"/>
 <instance part="R14" gate="G$1" x="129.54" y="93.98" rot="R90"/>
-<instance part="C7" gate="G$1" x="116.84" y="86.36"/>
 <instance part="C8" gate="G$1" x="147.32" y="83.82"/>
 <instance part="R15" gate="G$1" x="137.16" y="101.6" rot="R90"/>
@@
 <instance part="U$6" gate="G$1" x="177.8" y="185.42" rot="R180"/>
 <instance part="+3V5" gate="G$1" x="236.22" y="195.58"/>
+<instance part="SV1" gate="G$1" x="81.28" y="30.48" rot="R180"/>
+<instance part="GND7" gate="1" x="71.12" y="20.32"/>
 </instances>
 <busses>
@@
 <pinref part="R3" gate="G$1" pin="2"/>
 <wire x1="63.5" y1="170.18" x2="63.5" y2="177.8" width="0.1524" layer="91"/>
-<wire x1="63.5" y1="177.8" x2="50.8" y2="177.8" width="0.1524" layer="91"/>
-<pinref part="C1" gate="G$1" pin="1"/>
-<wire x1="50.8" y1="177.8" x2="50.8" y2="160.02" width="0.1524" layer="91"/>
 <pinref part="U$1" gate="G$1" pin="0"/>
-<wire x1="50.8" y1="177.8" x2="38.1" y2="177.8" width="0.1524" layer="91"/>
-<junction x="50.8" y="177.8"/>
+<wire x1="63.5" y1="177.8" x2="38.1" y2="177.8" width="0.1524" layer="91"/>
 </segment>
 </net>
@@
 <label x="86.36" y="165.1" size="1.778" layer="95"/>
 </segment>
+<segment>
+<pinref part="SV1" gate="G$1" pin="1"/>
+<wire x1="73.66" y1="35.56" x2="66.04" y2="35.56" width="0.1524" layer="91"/>
+<label x="60.96" y="35.56" size="1.778" layer="95"/>
+</segment>
 </net>
 <net name="N$4" class="0">
@@
 <pinref part="R6" gate="G$1" pin="2"/>
 <wire x1="63.5" y1="99.06" x2="63.5" y2="106.68" width="0.1524" layer="91"/>
-<wire x1="63.5" y1="106.68" x2="50.8" y2="106.68" width="0.1524" layer="91"/>
-<pinref part="C3" gate="G$1" pin="1"/>
-<wire x1="50.8" y1="106.68" x2="50.8" y2="88.9" width="0.1524" layer="91"/>
 <pinref part="U$2" gate="G$1" pin="0"/>
-<wire x1="50.8" y1="106.68" x2="38.1" y2="106.68" width="0.1524" layer="91"/>
-<junction x="50.8" y="106.68"/>
+<wire x1="63.5" y1="106.68" x2="38.1" y2="106.68" width="0.1524" layer="91"/>
 </segment>
 </net>
@@
 <pinref part="R10" gate="G$1" pin="2"/>
 <wire x1="127" y1="172.72" x2="127" y2="180.34" width="0.1524" layer="91"/>
-<wire x1="127" y1="180.34" x2="114.3" y2="180.34" width="0.1524" layer="91"/>
-<pinref part="C5" gate="G$1" pin="1"/>
-<wire x1="114.3" y1="180.34" x2="114.3" y2="162.56" width="0.1524" layer="91"/>
 <pinref part="U$3" gate="G$1" pin="0"/>
-<wire x1="114.3" y1="180.34" x2="101.6" y2="180.34" width="0.1524" layer="91"/>
-<junction x="114.3" y="180.34"/>
+<wire x1="127" y1="180.34" x2="101.6" y2="180.34" width="0.1524" layer="91"/>
 </segment>
 </net>
@@
 <pinref part="R14" gate="G$1" pin="2"/>
 <wire x1="129.54" y1="99.06" x2="129.54" y2="106.68" width="0.1524" layer="91"/>
-<wire x1="129.54" y1="106.68" x2="116.84" y2="106.68" width="0.1524" layer="91"/>
-<pinref part="C7" gate="G$1" pin="1"/>
-<wire x1="116.84" y1="106.68" x2="116.84" y2="88.9" width="0.1524" layer="91"/>
 <pinref part="U$4" gate="G$1" pin="0"/>
-<wire x1="116.84" y1="106.68" x2="104.14" y2="106.68" width="0.1524" layer="91"/>
-<junction x="116.84" y="106.68"/>
+<wire x1="129.54" y1="106.68" x2="104.14" y2="106.68" width="0.1524" layer="91"/>
 </segment>
 </net>
@@
 <label x="86.36" y="93.98" size="1.778" layer="95"/>
 </segment>
+<segment>
+<pinref part="SV1" gate="G$1" pin="2"/>
+<wire x1="73.66" y1="33.02" x2="66.04" y2="33.02" width="0.1524" layer="91"/>
+<label x="60.96" y="33.02" size="1.778" layer="95"/>
+</segment>
 </net>
 <net name="G4" class="0">
@@
 <label x="152.4" y="93.98" size="1.778" layer="95"/>
 </segment>
+<segment>
+<pinref part="SV1" gate="G$1" pin="4"/>
+<wire x1="73.66" y1="27.94" x2="66.04" y2="27.94" width="0.1524" layer="91"/>
+<label x="60.96" y="27.94" size="1.778" layer="95"/>
+</segment>
 </net>
 <net name="G3" class="0">
@@
 <label x="149.86" y="167.64" size="1.778" layer="95"/>
 </segment>
+<segment>
+<pinref part="SV1" gate="G$1" pin="3"/>
+<wire x1="73.66" y1="30.48" x2="66.04" y2="30.48" width="0.1524" layer="91"/>
+<label x="60.96" y="30.48" size="1.778" layer="95"/>
+</segment>
 </net>
 <net name="GND" class="0">
 <segment>
-<pinref part="C1" gate="G$1" pin="2"/>
-<wire x1="50.8" y1="152.4" x2="50.8" y2="137.16" width="0.1524" layer="91"/>
-<wire x1="50.8" y1="137.16" x2="63.5" y2="137.16" width="0.1524" layer="91"/>
 <pinref part="R2" gate="G$1" pin="1"/>
 <wire x1="63.5" y1="137.16" x2="63.5" y2="144.78" width="0.1524" layer="91"/>
@@
 <wire x1="81.28" y1="149.86" x2="81.28" y2="137.16" width="0.1524" layer="91"/>
 <wire x1="81.28" y1="137.16" x2="71.12" y2="137.16" width="0.1524" layer="91"/>
-<junction x="63.5" y="137.16"/>
 <pinref part="T1" gate="G$1" pin="E"/>
 <wire x1="71.12" y1="137.16" x2="66.04" y2="137.16" width="0.1524" layer="91"/>
@@
 </segment>
 <segment>
-<pinref part="C5" gate="G$1" pin="2"/>
-<wire x1="114.3" y1="154.94" x2="114.3" y2="139.7" width="0.1524" layer="91"/>
-<wire x1="114.3" y1="139.7" x2="127" y2="139.7" width="0.1524" layer="91"/>
 <pinref part="R9" gate="G$1" pin="1"/>
 <wire x1="127" y1="139.7" x2="127" y2="147.32" width="0.1524" layer="91"/>
@@
 <wire x1="144.78" y1="152.4" x2="144.78" y2="139.7" width="0.1524" layer="91"/>
 <wire x1="144.78" y1="139.7" x2="134.62" y2="139.7" width="0.1524" layer="91"/>
-<junction x="127" y="139.7"/>
 <pinref part="T3" gate="G$1" pin="E"/>
 <wire x1="134.62" y1="139.7" x2="129.54" y2="139.7" width="0.1524" layer="91"/>
@@
 </segment>
 <segment>
-<pinref part="C3" gate="G$1" pin="2"/>
-<wire x1="50.8" y1="81.28" x2="50.8" y2="66.04" width="0.1524" layer="91"/>
-<wire x1="50.8" y1="66.04" x2="63.5" y2="66.04" width="0.1524" layer="91"/>
 <pinref part="R5" gate="G$1" pin="1"/>
 <wire x1="63.5" y1="66.04" x2="63.5" y2="73.66" width="0.1524" layer="91"/>
@@
 <wire x1="81.28" y1="78.74" x2="81.28" y2="66.04" width="0.1524" layer="91"/>
 <wire x1="81.28" y1="66.04" x2="71.12" y2="66.04" width="0.1524" layer="91"/>
-<junction x="63.5" y="66.04"/>
 <pinref part="T2" gate="G$1" pin="E"/>
 <wire x1="71.12" y1="66.04" x2="66.04" y2="66.04" width="0.1524" layer="91"/>
@@
 </segment>
 <segment>
-<pinref part="C7" gate="G$1" pin="2"/>
-<wire x1="116.84" y1="81.28" x2="116.84" y2="66.04" width="0.1524" layer="91"/>
-<wire x1="116.84" y1="66.04" x2="129.54" y2="66.04" width="0.1524" layer="91"/>
 <pinref part="R13" gate="G$1" pin="1"/>
 <wire x1="129.54" y1="66.04" x2="129.54" y2="73.66" width="0.1524" layer="91"/>
@@
 <wire x1="147.32" y1="78.74" x2="147.32" y2="66.04" width="0.1524" layer="91"/>
 <wire x1="147.32" y1="66.04" x2="137.16" y2="66.04" width="0.1524" layer="91"/>
-<junction x="129.54" y="66.04"/>
 <pinref part="T4" gate="G$1" pin="E"/>
 <wire x1="137.16" y1="66.04" x2="132.08" y2="66.04" width="0.1524" layer="91"/>
@@
 <junction x="195.58" y="162.56"/>
 </segment>
-</net>
+<segment>
+<pinref part="SV1" gate="G$1" pin="5"/>
+<pinref part="GND7" gate="1" pin="GND"/>
+<wire x1="73.66" y1="25.4" x2="71.12" y2="25.4" width="0.1524" layer="91"/>
+<wire x1="71.12" y1="25.4" x2="71.12" y2="22.86" width="0.1524" layer="91"/>
+</segment>
+</net>

Commit message: Finished routing
Parts:
- added R19, R20, R21, R22: 100, resistor-power:RRS1/4
Connections:
- new net N$15: R20.2, SV1.2
- new net N$17: R21.2, SV1.3
- new net N$18: R22.2, SV1.4
- new net N$7: R19.2, SV1.1
- net G1: now also R22.1; no longer SV1.1
- net G2: now also R21.1; no longer SV1.2
- net G3: now also R20.1; no longer SV1.3
- net G4: now also R19.1; no longer SV1.4
Changed lines of the file:
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@@
 <part name="SV1" library="con-lsta" deviceset="FE05-1" device=""/>
 <part name="GND7" library="supply1" deviceset="GND" device=""/>
+<part name="R19" library="resistor-power" deviceset="R" device="RS1/4" value="100"/>
+<part name="R20" library="resistor-power" deviceset="R" device="RS1/4" value="100"/>
+<part name="R21" library="resistor-power" deviceset="R" device="RS1/4" value="100"/>
+<part name="R22" library="resistor-power" deviceset="R" device="RS1/4" value="100"/>
 </parts>
 <sheets>
@@
 <instance part="SV1" gate="G$1" x="81.28" y="30.48" rot="R180"/>
 <instance part="GND7" gate="1" x="71.12" y="20.32"/>
+<instance part="R19" gate="G$1" x="66.04" y="35.56"/>
+<instance part="R20" gate="G$1" x="66.04" y="33.02"/>
+<instance part="R21" gate="G$1" x="66.04" y="30.48"/>
+<instance part="R22" gate="G$1" x="66.04" y="27.94"/>
 </instances>
 <busses>
@@
 </segment>
 <segment>
-<pinref part="SV1" gate="G$1" pin="1"/>
-<wire x1="73.66" y1="35.56" x2="66.04" y2="35.56" width="0.1524" layer="91"/>
-<label x="60.96" y="35.56" size="1.778" layer="95"/>
+<pinref part="R22" gate="G$1" pin="1"/>
+<wire x1="60.96" y1="27.94" x2="58.42" y2="27.94" width="0.1524" layer="91"/>
+<label x="58.42" y="27.94" size="1.778" layer="95"/>
 </segment>
 </net>
@@
 </segment>
 <segment>
-<pinref part="SV1" gate="G$1" pin="2"/>
-<wire x1="73.66" y1="33.02" x2="66.04" y2="33.02" width="0.1524" layer="91"/>
-<label x="60.96" y="33.02" size="1.778" layer="95"/>
+<pinref part="R21" gate="G$1" pin="1"/>
+<wire x1="60.96" y1="30.48" x2="58.42" y2="30.48" width="0.1524" layer="91"/>
+<label x="58.42" y="30.48" size="1.778" layer="95"/>
 </segment>
 </net>
@@
 </segment>
 <segment>
-<pinref part="SV1" gate="G$1" pin="4"/>
-<wire x1="73.66" y1="27.94" x2="66.04" y2="27.94" width="0.1524" layer="91"/>
-<label x="60.96" y="27.94" size="1.778" layer="95"/>
+<pinref part="R19" gate="G$1" pin="1"/>
+<wire x1="60.96" y1="35.56" x2="58.42" y2="35.56" width="0.1524" layer="91"/>
+<label x="58.42" y="35.56" size="1.778" layer="95"/>
 </segment>
 </net>
@@
 </segment>
 <segment>
-<pinref part="SV1" gate="G$1" pin="3"/>
-<wire x1="73.66" y1="30.48" x2="66.04" y2="30.48" width="0.1524" layer="91"/>
-<label x="60.96" y="30.48" size="1.778" layer="95"/>
+<pinref part="R20" gate="G$1" pin="1"/>
+<wire x1="60.96" y1="33.02" x2="58.42" y2="33.02" width="0.1524" layer="91"/>
+<label x="58.42" y="33.02" size="1.778" layer="95"/>
 </segment>
 </net>
@@
 </segment>
 </net>
+<net name="N$7" class="0">
+<segment>
+<pinref part="SV1" gate="G$1" pin="1"/>
+<pinref part="R19" gate="G$1" pin="2"/>
+<wire x1="73.66" y1="35.56" x2="71.12" y2="35.56" width="0.1524" layer="91"/>
+</segment>
+</net>
+<net name="N$15" class="0">
+<segment>
+<pinref part="SV1" gate="G$1" pin="2"/>
+<pinref part="R20" gate="G$1" pin="2"/>
+<wire x1="73.66" y1="33.02" x2="71.12" y2="33.02" width="0.1524" layer="91"/>
+</segment>
+</net>
+<net name="N$17" class="0">
+<segment>
+<pinref part="SV1" gate="G$1" pin="3"/>
+<pinref part="R21" gate="G$1" pin="2"/>
+<wire x1="73.66" y1="30.48" x2="71.12" y2="30.48" width="0.1524" layer="91"/>
+</segment>
+</net>
+<net name="N$18" class="0">
+<segment>
+<pinref part="SV1" gate="G$1" pin="4"/>
+<pinref part="R22" gate="G$1" pin="2"/>
+<wire x1="73.66" y1="27.94" x2="71.12" y2="27.94" width="0.1524" layer="91"/>
+</segment>
+</net>
