File: Schematics/LOGIC/logic.brd (EAGLE design)
At the start: 54.6 x 50.3 mm, 10 parts

Commit message: Had to redo this board. Could not do 8mill traces on my mill
Parts:
- removed C3: (no value), SparkFun-Capacitors:CPOL-RADIAL-10UF-25V
- removed J1: (no value), SparkFun-Connectors:1X04_NO_SILK_ALL_ROUND
- removed R1: (no value), SparkFun-Resistors:AXIAL-0.4
- added JP1: (no value), pinhead:1X04
- moved JP2 10.2 mm to (15.1, 45.7), turned to 270 degrees
- moved JP3 2.55 mm to (15.0, 53.3), turned to 90 degrees
Connections:
- removed net PWM: R1.P$1, U$2.D6
- net AUDIO: now also U$2.D6; no longer C3.1, R1.P$2
- net GND: no longer C3.2
- net N$2: now also JP1.4; no longer J1.4
- net TUBE1: now also JP1.1; no longer J1.1
- net TUBE2: now also JP1.2; no longer J1.2
- net TUBE3: now also JP1.3; no longer J1.3
Routing:
- net GND: track 121.4 -> 106.4 mm
- net TUBE1: track 14.1 -> 10.4 mm
- net TUBE2: track 14.1 -> 10.4 mm
- net TUBE3: track 14.1 -> 10.4 mm
- net N$2: track 14.1 -> 10.4 mm
- net AUDIO: track 13.6 -> 10.3 mm
Changed lines of the file:
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@@
 </element>
 <element name="U$2" library="muon-tube" package="ESP12E_DEVKIT" value="ESP12E_DEVKIT" x="36.83" y="44.45" rot="R180"/>
-<element name="R1" library="SparkFun-Resistors" package="AXIAL-0.4" value="" x="20.447" y="41.91" rot="R270"/>
-<element name="C3" library="SparkFun-Capacitors" package="CPOL-RADIAL-10UF-25V" value="" x="15.875" y="42.164">
-<attribute name="PROD_ID" value="CAP-08440" x="15.875" y="42.164" size="1.778" layer="27" display="off"/>
-</element>
-<element name="JP2" library="pinhead" package="1X02" value="" x="14.605" y="35.56" rot="R90"/>
-<element name="JP3" library="pinhead" package="1X02" value="" x="14.732" y="50.8" rot="R270"/>
-<element name="J1" library="SparkFun-Connectors" package="1X04_NO_SILK_ALL_ROUND" value="" x="14.732" y="20.828" rot="R90">
-<attribute name="PROD_ID" value="CONN-09696" x="14.732" y="20.828" size="1.778" layer="27" rot="R90" display="off"/>
-</element>
+<element name="JP2" library="pinhead" package="1X02" value="" x="15.113" y="45.72" rot="R270"/>
+<element name="JP3" library="pinhead" package="1X02" value="" x="14.986" y="53.34" rot="R90"/>
+<element name="JP1" library="pinhead" package="1X04" value="" x="14.986" y="33.02" rot="R90"/>
 </elements>
 <signals>
@@
 <contactref element="U$2" pad="GND@1"/>
 <contactref element="U$2" pad="GND@3"/>
-<contactref element="C3" pad="2"/>
 <contactref element="U$2" pad="GND@0"/>
 <contactref element="U$2" pad="GND@2"/>
 <contactref element="JP2" pad="2"/>
 <contactref element="JP3" pad="2"/>
-<wire x1="59.055" y1="46.355" x2="59.055" y2="38.735" width="0.4064" layer="16"/>
-<wire x1="59.055" y1="38.735" x2="59.055" y2="33.02" width="0.4064" layer="16"/>
+<wire x1="59.055" y1="46.355" x2="59.055" y2="38.735" width="1.27" layer="16"/>
+<wire x1="59.055" y1="38.735" x2="59.055" y2="33.02" width="1.27" layer="16"/>
 <wire x1="59.055" y1="33.02" x2="58.42" y2="32.385" width="0.4064" layer="16"/>
 <wire x1="58.42" y1="32.385" x2="59.055" y2="32.385" width="0.4064" layer="16"/>
-<wire x1="59.055" y1="32.385" x2="60.96" y2="30.48" width="0.4064" layer="16"/>
-<wire x1="60.96" y1="30.48" x2="60.96" y2="24.13" width="0.4064" layer="16"/>
-<wire x1="59.055" y1="46.355" x2="55.88" y2="49.53" width="0.4064" layer="16"/>
-<wire x1="55.88" y1="49.53" x2="48.26" y2="49.53" width="0.4064" layer="16"/>
-<wire x1="25.4" y1="59.69" x2="38.1" y2="59.69" width="0.4064" layer="16"/>
-<wire x1="38.1" y1="59.69" x2="48.26" y2="59.69" width="0.4064" layer="16"/>
-<wire x1="48.26" y1="49.53" x2="40.64" y2="49.53" width="0.4064" layer="16"/>
-<wire x1="40.64" y1="49.53" x2="38.1" y2="52.07" width="0.4064" layer="16"/>
-<wire x1="38.1" y1="52.07" x2="38.1" y2="59.69" width="0.4064" layer="16"/>
-<wire x1="38.1" y1="52.07" x2="38.1" y2="48.514" width="0.4064" layer="16"/>
-<wire x1="38.1" y1="48.514" x2="31.496" y2="41.91" width="0.4064" layer="16"/>
-<wire x1="31.496" y1="41.91" x2="25.4" y2="41.91" width="0.4064" layer="16"/>
-<wire x1="14.732" y1="49.53" x2="14.732" y2="44.958" width="0.4064" layer="16"/>
-<wire x1="14.732" y1="44.958" x2="14.732" y2="42.291" width="0.4064" layer="16"/>
-<wire x1="14.732" y1="42.291" x2="14.605" y2="42.164" width="0.4064" layer="16"/>
-<wire x1="14.605" y1="42.164" x2="14.605" y2="36.83" width="0.4064" layer="16"/>
-<wire x1="25.4" y1="41.91" x2="22.606" y2="41.91" width="0.4064" layer="16"/>
-<wire x1="22.606" y1="41.91" x2="20.066" y2="44.45" width="0.4064" layer="16"/>
-<wire x1="20.066" y1="44.45" x2="15.24" y2="44.45" width="0.4064" layer="16"/>
-<wire x1="15.24" y1="44.45" x2="14.732" y2="44.958" width="0.4064" layer="16"/>
+<wire x1="59.055" y1="32.385" x2="60.96" y2="30.48" width="1.27" layer="16"/>
+<wire x1="60.96" y1="30.48" x2="60.96" y2="24.13" width="1.27" layer="16"/>
+<wire x1="59.055" y1="46.355" x2="55.88" y2="49.53" width="1.27" layer="16"/>
+<wire x1="55.88" y1="49.53" x2="48.26" y2="49.53" width="1.27" layer="16"/>
+<wire x1="14.986" y1="54.61" x2="14.986" y2="56.642" width="1.27" layer="16"/>
+<wire x1="14.986" y1="56.642" x2="18.034" y2="59.69" width="1.27" layer="16"/>
+<wire x1="18.034" y1="59.69" x2="25.4" y2="59.69" width="1.27" layer="16"/>
+<wire x1="15.113" y1="44.45" x2="15.113" y2="43.561" width="1.27" layer="16"/>
+<wire x1="15.113" y1="43.561" x2="16.764" y2="41.91" width="1.27" layer="16"/>
+<wire x1="16.764" y1="41.91" x2="25.4" y2="41.91" width="1.27" layer="16"/>
+<wire x1="25.4" y1="59.69" x2="36.576" y2="59.69" width="1.27" layer="16"/>
+<wire x1="36.576" y1="59.69" x2="48.26" y2="59.69" width="1.27" layer="16"/>
+<wire x1="48.26" y1="49.53" x2="36.83" y2="49.53" width="1.27" layer="16"/>
+<wire x1="36.83" y1="49.53" x2="36.576" y2="49.53" width="1.27" layer="16"/>
+<wire x1="36.576" y1="59.69" x2="36.576" y2="49.784" width="1.27" layer="16"/>
+<wire x1="36.576" y1="49.784" x2="36.83" y2="49.53" width="1.27" layer="16"/>
+<wire x1="15.113" y1="44.45" x2="14.986" y2="54.61" width="0" layer="19" extent="1-1"/>
 </signal>
 <signal name="N$1">
@@
 <contactref element="C1" pad="1"/>
 <contactref element="U2" pad="IN"/>
-<wire x1="55.88" y1="24.13" x2="55.88" y2="32.385" width="0.4064" layer="16"/>
-<wire x1="55.88" y1="32.385" x2="55.88" y2="38.1" width="0.4064" layer="16"/>
+<wire x1="55.88" y1="24.13" x2="55.88" y2="32.385" width="1.27" layer="16"/>
+<wire x1="55.88" y1="32.385" x2="55.88" y2="38.1" width="1.27" layer="16"/>
 <wire x1="55.88" y1="38.1" x2="56.515" y2="38.735" width="0.4064" layer="16"/>
 </signal>
@@
 <contactref element="C2" pad="1"/>
 <contactref element="U$2" pad="VIN"/>
-<wire x1="61.595" y1="46.355" x2="61.595" y2="56.515" width="0.4064" layer="16"/>
-<wire x1="61.595" y1="56.515" x2="55.88" y2="62.23" width="0.4064" layer="16"/>
-<wire x1="55.88" y1="62.23" x2="48.26" y2="62.23" width="0.4064" layer="16"/>
-<wire x1="61.595" y1="46.355" x2="61.595" y2="38.735" width="0.4064" layer="16"/>
+<wire x1="61.595" y1="46.355" x2="61.595" y2="56.515" width="1.27" layer="16"/>
+<wire x1="61.595" y1="56.515" x2="55.88" y2="62.23" width="1.27" layer="16"/>
+<wire x1="55.88" y1="62.23" x2="48.26" y2="62.23" width="1.27" layer="16"/>
+<wire x1="61.595" y1="46.355" x2="61.595" y2="38.735" width="1.27" layer="16"/>
 </signal>
 <signal name="TUBE1">
 <contactref element="U$2" pad="D1"/>
-<contactref element="J1" pad="1"/>
-<wire x1="25.4" y1="29.21" x2="24.384" y2="29.21" width="0.4064" layer="16"/>
-<wire x1="24.384" y1="29.21" x2="23.114" y2="27.94" width="0.4064" layer="16"/>
-<wire x1="23.114" y1="27.94" x2="21.844" y2="27.94" width="0.4064" layer="16"/>
-<wire x1="21.844" y1="27.94" x2="14.732" y2="20.828" width="0.4064" layer="16"/>
+<contactref element="JP1" pad="1"/>
+<wire x1="25.4" y1="29.21" x2="14.986" y2="29.21" width="1.27" layer="16"/>
 </signal>
 <signal name="TUBE2">
 <contactref element="U$2" pad="D2"/>
-<contactref element="J1" pad="2"/>
-<wire x1="25.4" y1="31.75" x2="24.384" y2="31.75" width="0.4064" layer="16"/>
-<wire x1="24.384" y1="31.75" x2="22.352" y2="29.718" width="0.4064" layer="16"/>
-<wire x1="22.352" y1="29.718" x2="21.082" y2="29.718" width="0.4064" layer="16"/>
-<wire x1="21.082" y1="29.718" x2="14.732" y2="23.368" width="0.4064" layer="16"/>
+<contactref element="JP1" pad="2"/>
+<wire x1="25.4" y1="31.75" x2="14.986" y2="31.75" width="1.27" layer="16"/>
 </signal>
 <signal name="TUBE3">
 <contactref element="U$2" pad="D3"/>
-<contactref element="J1" pad="3"/>
-<wire x1="25.4" y1="34.29" x2="24.13" y2="34.29" width="0.4064" layer="16"/>
-<wire x1="24.13" y1="34.29" x2="21.336" y2="31.496" width="0.4064" layer="16"/>
-<wire x1="21.336" y1="31.496" x2="20.32" y2="31.496" width="0.4064" layer="16"/>
-<wire x1="20.32" y1="31.496" x2="14.732" y2="25.908" width="0.4064" layer="16"/>
+<contactref element="JP1" pad="3"/>
+<wire x1="25.4" y1="34.29" x2="14.986" y2="34.29" width="1.27" layer="16"/>
 </signal>
 <signal name="GATE">
 <contactref element="JP3" pad="1"/>
 <contactref element="U$2" pad="D8"/>
-<wire x1="25.4" y1="52.07" x2="14.732" y2="52.07" width="0.4064" layer="16"/>
+<wire x1="25.4" y1="52.07" x2="14.986" y2="52.07" width="1.27" layer="16"/>
 </signal>
 <signal name="AUDIO">
-<contactref element="R1" pad="P$2"/>
-<contactref element="C3" pad="1"/>
 <contactref element="JP2" pad="1"/>
-<wire x1="14.605" y1="34.29" x2="17.907" y2="34.29" width="0.4064" layer="16"/>
-<wire x1="17.907" y1="34.29" x2="20.447" y2="36.83" width="0.4064" layer="16"/>
-<wire x1="20.447" y1="36.83" x2="20.447" y2="38.862" width="0.4064" layer="16"/>
-<wire x1="20.447" y1="38.862" x2="17.145" y2="42.164" width="0.4064" layer="16"/>
-</signal>
-<signal name="PWM">
 <contactref element="U$2" pad="D6"/>
-<contactref element="R1" pad="P$1"/>
-<wire x1="25.4" y1="46.99" x2="20.447" y2="46.99" width="0" layer="19" extent="1-16"/>
+<wire x1="25.4" y1="46.99" x2="15.113" y2="46.99" width="1.27" layer="16"/>
 </signal>
 <signal name="N$2">
 <contactref element="U$2" pad="D4"/>
-<contactref element="J1" pad="4"/>
-<wire x1="25.4" y1="36.83" x2="24.384" y2="36.83" width="0.4064" layer="16"/>
-<wire x1="24.384" y1="36.83" x2="20.574" y2="33.02" width="0.4064" layer="16"/>
-<wire x1="20.574" y1="33.02" x2="19.304" y2="33.02" width="0.4064" layer="16"/>
-<wire x1="19.304" y1="33.02" x2="14.732" y2="28.448" width="0.4064" layer="16"/>
+<contactref element="JP1" pad="4"/>
+<wire x1="25.4" y1="36.83" x2="14.986" y2="36.83" width="1.27" layer="16"/>
 </signal>
 </signals>
