File: Schematics/LOGIC/logic.sch (EAGLE design)
At the start: 10 parts

Commit message: Had to redo this board. Could not do 8mill traces on my mill
Parts:
- removed C3: (no value), SparkFun-Capacitors:10UF-25V-20%(PTH)
- removed J1: (no value), SparkFun-Connectors:M04NO_SILK_ALL_ROUND
- removed R1: (no value), SparkFun-Resistors:RESISTORPTH-1/4W
- added JP1: (no value), pinhead:PINHD-1X4
Connections:
- removed net PWM: R1.1, U$2.D6
- net AUDIO: now also U$2.D6; no longer C3.+, R1.2
- net GND: no longer C3.-
- net N$2: now also JP1.4; no longer J1.4
- net TUBE1: now also JP1.1; no longer J1.1
- net TUBE2: now also JP1.2; no longer J1.2
- net TUBE3: now also JP1.3; no longer J1.3
Changed lines of the file:
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@@
 <part name="U$2" library="muon-tube" deviceset="ESP12E_DEVKIT" device=""/>
 <part name="GND3" library="SparkFun-Aesthetics" deviceset="GND" device=""/>
-<part name="R1" library="SparkFun-Resistors" deviceset="RESISTOR" device="PTH-1/4W"/>
-<part name="C3" library="SparkFun-Capacitors" deviceset="10UF-25V-20%(PTH)" device=""/>
-<part name="GND4" library="SparkFun-Aesthetics" deviceset="GND" device=""/>
 <part name="JP2" library="pinhead" deviceset="PINHD-1X2" device=""/>
 <part name="JP3" library="pinhead" deviceset="PINHD-1X2" device=""/>
 <part name="GND5" library="SparkFun-Aesthetics" deviceset="GND" device=""/>
-<part name="J1" library="SparkFun-Connectors" deviceset="M04" device="NO_SILK_ALL_ROUND"/>
+<part name="JP1" library="pinhead" deviceset="PINHD-1X4" device=""/>
 </parts>
 <sheets>
@@
 <instance part="U$2" gate="G$1" x="50.8" y="154.94"/>
 <instance part="GND3" gate="1" x="73.66" y="132.08"/>
-<instance part="R1" gate="G$1" x="91.44" y="152.4"/>
-<instance part="C3" gate="G$1" x="99.06" y="149.86"/>
-<instance part="GND4" gate="1" x="99.06" y="139.7"/>
 <instance part="JP2" gate="G$1" x="142.24" y="137.16"/>
 <instance part="JP3" gate="G$1" x="142.24" y="121.92"/>
 <instance part="GND5" gate="1" x="132.08" y="106.68"/>
-<instance part="J1" gate="G$1" x="149.86" y="167.64" rot="R180"/>
+<instance part="JP1" gate="A" x="147.32" y="165.1"/>
 </instances>
 <busses>
@@
 <wire x1="73.66" y1="157.48" x2="73.66" y2="139.7" width="0.1524" layer="91"/>
 <junction x="73.66" y="139.7"/>
-</segment>
-<segment>
-<pinref part="C3" gate="G$1" pin="-"/>
-<pinref part="GND4" gate="1" pin="GND"/>
-<wire x1="99.06" y1="144.78" x2="99.06" y2="142.24" width="0.1524" layer="91"/>
 </segment>
 <segment>
@@
 <label x="71.12" y="170.18" size="1.778" layer="95"/>
 <wire x1="68.58" y1="170.18" x2="144.78" y2="170.18" width="0.1524" layer="91"/>
-<pinref part="J1" gate="G$1" pin="1"/>
+<pinref part="JP1" gate="A" pin="1"/>
 </segment>
 </net>
@@
 <label x="71.12" y="167.64" size="1.778" layer="95"/>
 <wire x1="144.78" y1="167.64" x2="68.58" y2="167.64" width="0.1524" layer="91"/>
-<pinref part="J1" gate="G$1" pin="2"/>
+<pinref part="JP1" gate="A" pin="2"/>
 </segment>
 </net>
@@
 <label x="71.12" y="165.1" size="1.778" layer="95"/>
 <wire x1="68.58" y1="165.1" x2="144.78" y2="165.1" width="0.1524" layer="91"/>
-<pinref part="J1" gate="G$1" pin="3"/>
+<pinref part="JP1" gate="A" pin="3"/>
 </segment>
 </net>
@@
 <net name="AUDIO" class="0">
 <segment>
-<pinref part="R1" gate="G$1" pin="2"/>
-<pinref part="C3" gate="G$1" pin="+"/>
-<wire x1="96.52" y1="152.4" x2="99.06" y2="152.4" width="0.1524" layer="91"/>
-<wire x1="99.06" y1="152.4" x2="106.68" y2="152.4" width="0.1524" layer="91"/>
-<junction x="99.06" y="152.4"/>
-<label x="99.06" y="152.4" size="1.778" layer="95"/>
-</segment>
-<segment>
 <pinref part="JP2" gate="G$1" pin="1"/>
 <wire x1="139.7" y1="139.7" x2="119.38" y2="139.7" width="0.1524" layer="91"/>
 <label x="119.38" y="139.7" size="1.778" layer="95"/>
 </segment>
-</net>
-<net name="PWM" class="0">
 <segment>
 <pinref part="U$2" gate="G$1" pin="D6"/>
-<pinref part="R1" gate="G$1" pin="1"/>
 <wire x1="68.58" y1="152.4" x2="86.36" y2="152.4" width="0.1524" layer="91"/>
 <label x="81.28" y="152.4" size="1.778" layer="95"/>
@@
 <segment>
 <pinref part="U$2" gate="G$1" pin="D4"/>
-<pinref part="J1" gate="G$1" pin="4"/>
 <wire x1="68.58" y1="162.56" x2="144.78" y2="162.56" width="0.1524" layer="91"/>
+<pinref part="JP1" gate="A" pin="4"/>
 </segment>
 </net>
